Commit message: Se agrega un archivo .launch para visualizar el robot el gazebo

File: urdf/kobuki.urdf (robot description, URDF)
Before this commit: robot kobuki_v1, 6 links, 5 joints
Joints:
- joint sphere_joint2: origin xyz=-0.115 0.0 0.007 rpy=0.0 0.0 0.0 -> xyz=-0.115 0.0 0.009 rpy=0.0 0.0 0.0

Commit message: Se agregan los nodos de python para teleoperacion

File: urdf/kobuki.urdf (robot description, URDF)
Before this commit: robot kobuki_v1, 6 links, 5 joints
Joints:
- joint joint_left: limit effort=10 velocity=6.0 -> effort=20 velocity=20.0
- joint joint_right: limit effort=10 velocity=6.0 -> effort=20 velocity=20.0
